Commit message: rename prefix to tf_prefix

File: urdf/rbs_gripper.xacro (robot description, xacro)
@@ -4,5 +4,5 @@
   <xacro:arg name="hardware" default="gazebo"/>
   <link name="world"/>
-  <xacro:rbs_gripper prefix="" gripper_name="rbs-gripper" parent="world" hardware="$(arg hardware)">
+  <xacro:rbs_gripper tf_prefix="" gripper_name="rbs-gripper" parent="world" hardware="$(arg hardware)">
     <origin xyz="0.0 0.0 0.0" rpy="0.0 0.0 0.0"/>
   </xacro:rbs_gripper>

File: urdf/rbs_gripper_macro.xacro (robot description, xacro)
@@ -2,13 +2,13 @@
 <robot xmlns:xacro="http://wiki.ros.org/xacro">
   <xacro:include filename="$(find rbs_gripper)/urdf/rbs_gripper_ros2_control.xacro" />
-  <xacro:macro name="rbs_gripper" params="prefix gripper_name *origin parent hardware">
-    <xacro:rbs_gripper_hardware prefix="${prefix}" gripper_name="${gripper_name}"
+  <xacro:macro name="rbs_gripper" params="tf_prefix gripper_name *origin parent hardware">
+    <xacro:rbs_gripper_hardware tf_prefix="${tf_prefix}" gripper_name="${gripper_name}"
       hardware="${hardware}" />
-    <joint name="${prefix}${gripper_name}_gripper_base_joint" type="fixed">
+    <joint name="${tf_prefix}${gripper_name}_gripper_base_joint" type="fixed">
       <origin xyz="0 0 0" rpy="0 0 0" />
       <parent link="${parent}" />
-      <child link="${prefix}${gripper_name}_gripper_base_link" />
+      <child link="${tf_prefix}${gripper_name}_gripper_base_link" />
     </joint>
-    <link name="${prefix}${gripper_name}_gripper_base_link">
+    <link name="${tf_prefix}${gripper_name}_gripper_base_link">
       <inertial>
         <origin xyz="0.000364704367134063 0.0336387482840125 0.0593891203954369" rpy="0 0 0" />
@@ -22,5 +22,5 @@
           <mesh filename="file://$(find rbs_gripper)/meshes/visual/Grip_Base.dae" />
         </geometry>
-        <material name="${prefix}${gripper_name}_material">
+        <material name="${tf_prefix}${gripper_name}_material">
           <color rgba="0.752941176470588 0.752941176470588 0.752941176470588 1" />
         </material>
@@ -33,5 +33,5 @@
       </collision>
     </link>
-    <link name="${prefix}${gripper_name}_rot_base_link">
+    <link name="${tf_prefix}${gripper_name}_rot_base_link">
       <inertial>
         <origin xyz="6.79110135283868E-11 -3.80956832067611E-10 0.00775394473595793" rpy="0 0 0" />
@@ -45,5 +45,5 @@
           <mesh filename="file://$(find rbs_gripper)/meshes/visual/Grip_Rotator.dae" />
         </geometry>
-        <material name="${prefix}${gripper_name}_material">
+        <material name="${tf_prefix}${gripper_name}_material">
           <color rgba="0.250980392156863 0.250980392156863 0.250980392156863 1" />
         </material>
@@ -56,13 +56,13 @@
       </collision>
     </link>
-    <joint name="${prefix}${gripper_name}_rot_base_joint" type="revolute">
+    <joint name="${tf_prefix}${gripper_name}_rot_base_joint" type="revolute">
       <origin xyz="0 0 0.10861" rpy="0 0 0" />
-      <parent link="${prefix}${gripper_name}_gripper_base_link" />
-      <child link="${prefix}${gripper_name}_rot_base_link" />
+      <parent link="${tf_prefix}${gripper_name}_gripper_base_link" />
+      <child link="${tf_prefix}${gripper_name}_rot_base_link" />
       <axis xyz="0 0 1" />
       <limit lower="-3.14159" upper="3.14159" effort="78" velocity="0.52" />
     <dynamics damping="0" friction="0"/>
     </joint>
-    <link name="${prefix}${gripper_name}_l_finger_link">
+    <link name="${tf_prefix}${gripper_name}_l_finger_link">
       <inertial>
         <origin xyz="0.00399878118534129 0.0187296413885176 -0.0777776233934166" rpy="0 0 0" />
@@ -76,5 +76,5 @@
           <mesh filename="file://$(find rbs_gripper)/meshes/visual/Gripper_1.dae" />
         </geometry>
-        <material name="${prefix}${gripper_name}_material">
+        <material name="${tf_prefix}${gripper_name}_material">
           <color rgba="0.752941176470588 0 0 1" />
         </material>
@@ -87,13 +87,13 @@
       </collision>
     </link>
-    <joint name="${prefix}${gripper_name}_l_finger_joint" type="prismatic">
+    <joint name="${tf_prefix}${gripper_name}_l_finger_joint" type="prismatic">
       <origin xyz="0 0 0.1071" rpy="0 0 1.5708" />
-      <parent link="${prefix}${gripper_name}_rot_base_link" />
-      <child link="${prefix}${gripper_name}_l_finger_link" />
+      <parent link="${tf_prefix}${gripper_name}_rot_base_link" />
+      <child link="${tf_prefix}${gripper_name}_l_finger_link" />
       <axis xyz="-1 0 0" />
       <limit lower="0" upper="0.064" effort="10" velocity="0.53" />
-			<mimic joint="${prefix}${gripper_name}_r_finger_joint" multiplier="1" />
+			<mimic joint="${tf_prefix}${gripper_name}_r_finger_joint" multiplier="1" />
     </joint>
-    <link name="${prefix}${gripper_name}_r_finger_link">
+    <link name="${tf_prefix}${gripper_name}_r_finger_link">
       <inertial>
         <origin xyz="0.0039988 -0.077778 -0.01873" rpy="0 0 0" />
@@ -108,5 +108,5 @@
           <mesh filename="file://$(find rbs_gripper)/meshes/visual/Gripper_2.dae" />
         </geometry>
-        <material name="${prefix}${gripper_name}_material">
+        <material name="${tf_prefix}${gripper_name}_material">
           <color rgba="0.75294 0 0 1" />
         </material>
@@ -119,16 +119,16 @@
       </collision>
     </link>
-    <joint name="${prefix}${gripper_name}_r_finger_joint" type="prismatic">
+    <joint name="${tf_prefix}${gripper_name}_r_finger_joint" type="prismatic">
       <origin xyz="0 0 0.1071" rpy="1.5708 0 -1.5708" />
-      <parent link="${prefix}${gripper_name}_rot_base_link" />
-      <child link="${prefix}${gripper_name}_r_finger_link" />
+      <parent link="${tf_prefix}${gripper_name}_rot_base_link" />
+      <child link="${tf_prefix}${gripper_name}_r_finger_link" />
       <axis xyz="-1 0 0" />
       <limit lower="0" upper="0.064" effort="10" velocity="0.53" />
     </joint>
-    <link name="${prefix}gripper_grasp_point" />
-    <joint name="${prefix}${gripper_name}_gripper_tool0_joint" type="fixed">
+    <link name="${tf_prefix}gripper_grasp_point" />
+    <joint name="${tf_prefix}${gripper_name}_gripper_tool0_joint" type="fixed">
       <origin xyz="0 0 0.09139" rpy="0 0 0" />
-      <parent link="${prefix}${gripper_name}_rot_base_link" />
-      <child link="${prefix}gripper_grasp_point" />
+      <parent link="${tf_prefix}${gripper_name}_rot_base_link" />
+      <child link="${tf_prefix}gripper_grasp_point" />
     </joint>
   </xacro:macro>

File: urdf/rbs_gripper_ros2_control.xacro (robot description, xacro)
@@ -2,6 +2,6 @@
 <robot xmlns:xacro="http://www.ros.org/wiki/xacro">
   <xacro:macro name="rbs_gripper_hardware"
-    params="prefix gripper_name hardware">
-    <ros2_control name="${prefix}${gripper_name}_${hardware}" type="system">
+    params="tf_prefix gripper_name hardware">
+    <ros2_control name="${tf_prefix}${gripper_name}_${hardware}" type="system">
       <!-- Plugins -->
       <hardware>
@@ -19,5 +19,5 @@
       </hardware>
       <!-- Joint interfaces -->
-      <joint name="${prefix}${gripper_name}_rot_base_joint">
+      <joint name="${tf_prefix}${gripper_name}_rot_base_joint">
         <xacro:if value="${hardware=='gazebo'}">
           <state_interface name="position">
@@ -33,5 +33,5 @@
         <state_interface name="effort" />
       </joint>
-      <joint name="${prefix}${gripper_name}_r_finger_joint">
+      <joint name="${tf_prefix}${gripper_name}_r_finger_joint">
         <!-- With Gazebo, we have mimic joints, so we only need this command interface
                 activated -->
@@ -49,6 +49,6 @@
         <state_interface name="effort" />
       </joint>
-      <joint name="${prefix}${gripper_name}_l_finger_joint">
-        <param name="mimic">${prefix}${gripper_name}_r_finger_joint</param>
+      <joint name="${tf_prefix}${gripper_name}_l_finger_joint">
+        <param name="mimic">${tf_prefix}${gripper_name}_r_finger_joint</param>
         <param name="multiplier">1</param>
         <xacro:unless value="${hardware == 'gazebo'}">
