Commit message: fix for simulation

File: urdf/rbs_gripper_macro.xacro (robot description, xacro)
@@ -61,5 +61,6 @@
       <child link="${prefix}${gripper_name}_rot_base_link" />
       <axis xyz="0 0 1" />
-      <limit lower="0" upper="0" effort="0" velocity="0" />
+      <limit lower="-3.14159" upper="3.14159" effort="78" velocity="0.52" />
+    <dynamics damping="0" friction="0"/>
     </joint>
     <link name="${prefix}${gripper_name}_l_finger_link">
@@ -91,5 +92,5 @@
       <child link="${prefix}${gripper_name}_l_finger_link" />
       <axis xyz="-1 0 0" />
-      <limit lower="0" upper="0.064" effort="0" velocity="0" />
+      <limit lower="0" upper="0.064" effort="10" velocity="0.53" />
 			<mimic joint="${prefix}${gripper_name}_r_finger_joint" multiplier="1" />
     </joint>
@@ -123,10 +124,10 @@
       <child link="${prefix}${gripper_name}_r_finger_link" />
       <axis xyz="-1 0 0" />
-      <limit lower="0" upper="0.064" effort="0" velocity="0" />
+      <limit lower="0" upper="0.064" effort="10" velocity="0.53" />
     </joint>
     <link name="${prefix}gripper_grasp_point" />
     <joint name="${prefix}${gripper_name}_gripper_tool0_joint" type="fixed">
-      <origin xyz="0 0 0.2" rpy="0 0 0" />
-      <parent link="${prefix}${parent}" />
+      <origin xyz="0 0 0.09139" rpy="0 0 0" />
+      <parent link="${prefix}${gripper_name}_rot_base_link" />
       <child link="${prefix}gripper_grasp_point" />
     </joint>

File: urdf/rbs_gripper_ros2_control.xacro (robot description, xacro)
@@ -31,4 +31,5 @@
         <command_interface name="position" />
         <state_interface name="velocity" />
+        <state_interface name="effort" />
       </joint>
       <joint name="${prefix}${gripper_name}_r_finger_joint">
@@ -46,4 +47,5 @@
         <command_interface name="position" />
         <state_interface name="velocity" />
+        <state_interface name="effort" />
       </joint>
       <joint name="${prefix}${gripper_name}_l_finger_joint">
@@ -54,4 +56,5 @@
           <state_interface name="position" />
           <state_interface name="velocity" />
+          <state_interface name="effort" />
         </xacro:unless>
       </joint>

Commit message: update for compatibility with rbs framework

File: urdf/rbs_gripper_macro.xacro (robot description, xacro)
@@ -20,5 +20,5 @@
         <origin xyz="0 0 0" rpy="0 0 0" />
         <geometry>
-          <mesh filename="file://$(find rbs_gripper)/meshes/visual/Grip_Base.dae" />
+          <mesh filename="file://$(find rbs_gripper)/meshes/visual/base.dae" />
         </geometry>
         <material name="${tf_prefix}${gripper_name}_material">
@@ -29,5 +29,5 @@
         <origin xyz="0 0 0" rpy="0 0 0" />
         <geometry>
-          <mesh filename="file://$(find rbs_gripper)/meshes/collision/Grip_Base.stl" />
+          <mesh filename="file://$(find rbs_gripper)/meshes/collision/base.stl" />
         </geometry>
       </collision>
@@ -43,5 +43,5 @@
         <origin xyz="0 0 0" rpy="0 0 0" />
         <geometry>
-          <mesh filename="file://$(find rbs_gripper)/meshes/visual/Grip_Rotator.dae" />
+          <mesh filename="file://$(find rbs_gripper)/meshes/visual/rotor.dae" />
         </geometry>
         <material name="${tf_prefix}${gripper_name}_material">
@@ -52,5 +52,5 @@
         <origin xyz="0 0 0" rpy="0 0 0" />
         <geometry>
-          <mesh filename="file://$(find rbs_gripper)/meshes/collision/Grip_Rotator.stl" />
+          <mesh filename="file://$(find rbs_gripper)/meshes/collision/rotor.stl" />
         </geometry>
       </collision>
@@ -62,5 +62,4 @@
       <axis xyz="0 0 1" />
       <limit lower="-3.14159" upper="3.14159" effort="78" velocity="0.52" />
-    <dynamics damping="0" friction="0"/>
     </joint>
     <link name="${tf_prefix}${gripper_name}_l_finger_link">
@@ -74,5 +73,5 @@
         <origin xyz="0 0 0" rpy="0 0 0" />
         <geometry>
-          <mesh filename="file://$(find rbs_gripper)/meshes/visual/Gripper_1.dae" />
+          <mesh filename="file://$(find rbs_gripper)/meshes/visual/finger.dae" />
         </geometry>
         <material name="${tf_prefix}${gripper_name}_material">
@@ -83,5 +82,5 @@
         <origin xyz="0 0 0" rpy="0 0 0" />
         <geometry>
-          <mesh filename="file://$(find rbs_gripper)/meshes/collision/Gripper_1.stl" />
+          <mesh filename="file://$(find rbs_gripper)/meshes/collision/finger.stl" />
         </geometry>
       </collision>
@@ -106,5 +105,5 @@
         <origin xyz="0 0 0" rpy="0 0 0" />
         <geometry>
-          <mesh filename="file://$(find rbs_gripper)/meshes/visual/Gripper_2.dae" />
+          <mesh filename="file://$(find rbs_gripper)/meshes/visual/finger.dae" />
         </geometry>
         <material name="${tf_prefix}${gripper_name}_material">
@@ -115,10 +114,10 @@
         <origin xyz="0 0 0" rpy="0 0 0" />
         <geometry>
-          <mesh filename="file://$(find rbs_gripper)/meshes/collision/Gripper_2.stl" />
+          <mesh filename="file://$(find rbs_gripper)/meshes/collision/finger.stl" />
         </geometry>
       </collision>
     </link>
     <joint name="${tf_prefix}${gripper_name}_r_finger_joint" type="prismatic">
-      <origin xyz="0 0 0.1071" rpy="1.5708 0 -1.5708" />
+      <origin xyz="0 0 0.1071" rpy="0 0 -1.5708" />
       <parent link="${tf_prefix}${gripper_name}_rot_base_link" />
       <child link="${tf_prefix}${gripper_name}_r_finger_link" />

File: urdf/rbs_gripper_ros2_control.xacro (robot description, xacro)
@@ -30,4 +30,6 @@
         </xacro:unless>
         <command_interface name="position" />
+        <command_interface name="velocity"/>
+        <command_interface name="effort"/>
         <state_interface name="velocity" />
         <state_interface name="effort" />
@@ -38,5 +40,5 @@
         <xacro:if value="${hardware=='gazebo'}">
           <state_interface name="position">
-            <param name="initial_value">0.004</param>
+            <param name="initial_value">0.000</param>
           </state_interface>
         </xacro:if>
@@ -46,4 +48,6 @@
         </xacro:unless>
         <command_interface name="position" />
+        <command_interface name="velocity"/>
+        <command_interface name="effort"/>
         <state_interface name="velocity" />
         <state_interface name="effort" />
@@ -54,4 +58,6 @@
         <xacro:unless value="${hardware == 'gazebo'}">
           <command_interface name="position" />
+          <command_interface name="velocity"/>
+          <command_interface name="effort"/>
           <state_interface name="position" />
           <state_interface name="velocity" />
