Commit message: remove effort states

File: urdf/rbs_gripper.urdf (robot description, URDF)
Before this commit: robot rbs-gripper-description, 3 links, 3 joints
Links:
- removed link finger
- added link finger_1, mass 0.0601996441483964; collision mesh filename=/home/narmak/rbs_ws/install/rbs_gripper/share/rbs_gripper/m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; visual mesh filename=/home/narmak/rbs_ws/install/rbs_gripper/share/rbs_gripper/m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
- added link finger_2, mass 0.0602; collision mesh filename=/home/narmak/rbs_ws/install/rbs_gripper/share/rbs_gripper/m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; visual mesh filename=/home/narmak/rbs_ws/install/rbs_gripper/share/rbs_gripper/m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
- link base: geometry collision mesh filename=/home/narmak/rbs_ws/install/rbs_gripper/share/rbs_gripper/m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; visual mesh filename=/home/narmak/rbs_ws/install/rbs_gripper/share/rbs_gripper/m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
- link rotor: geometry collision mesh filename=/home/narmak/rbs_ws/install/rbs_gripper/share/rbs_gripper/m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; visual mesh filename=/home/narmak/rbs_ws/install/rbs_gripper/share/rbs_gripper/m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
Joints:
- joint open_1: child finger -> finger_1; mimic (none) -> joint=finger_2 multiplier=1
- joint open_2: child finger -> finger_2

File: urdf/rbs_gripper_macro.xacro (robot description, xacro)
@@ -2,4 +2,5 @@
 <robot xmlns:xacro="http://wiki.ros.org/xacro">
   <xacro:include filename="$(find rbs_gripper)/urdf/rbs_gripper_ros2_control.xacro" />
+  <xacro:include filename="$(find rbs_gripper)/urdf/gazebos_macro.xacro"/>
   <xacro:macro name="rbs_gripper" params="tf_prefix gripper_name *origin parent hardware">
     <xacro:rbs_gripper_hardware tf_prefix="${tf_prefix}" gripper_name="${gripper_name}"
@@ -131,4 +132,7 @@
       <child link="${tf_prefix}gripper_grasp_point" />
     </joint>
+    <!-- <xacro:rbs_griper_gazebo_stuff link_name="${tf_prefix}${gripper_name}_rot_base_link"/> -->
+    <!-- <xacro:rbs_griper_gazebo_stuff link_name="${tf_prefix}${gripper_name}_l_finger_link"/> -->
+    <!-- <xacro:rbs_griper_gazebo_stuff link_name="${tf_prefix}${gripper_name}_r_finger_link"/> -->
   </xacro:macro>
 </robot>

File: urdf/rbs_gripper_ros2_control.xacro (robot description, xacro)
@@ -1,4 +1,5 @@
 <?xml version="1.0"?>
 <robot xmlns:xacro="http://www.ros.org/wiki/xacro">
+  <xacro:include filename="$(find rbs_gripper)/urdf/transmission_macro.xacro"/>
   <xacro:macro name="rbs_gripper_hardware"
     params="tf_prefix gripper_name hardware">
@@ -31,7 +32,7 @@
         <command_interface name="position" />
         <command_interface name="velocity"/>
-        <command_interface name="effort"/>
+        <!-- <command_interface name="acceleration"/> -->
         <state_interface name="velocity" />
-        <state_interface name="effort" />
+        <!-- <state_interface name="acceleration" /> -->
       </joint>
       <joint name="${tf_prefix}${gripper_name}_r_finger_joint">
@@ -40,5 +41,5 @@
         <xacro:if value="${hardware=='gazebo'}">
           <state_interface name="position">
-            <param name="initial_value">0.000</param>
+            <param name="initial_value">0.004</param>
           </state_interface>
         </xacro:if>
@@ -49,7 +50,7 @@
         <command_interface name="position" />
         <command_interface name="velocity"/>
-        <command_interface name="effort"/>
+        <!-- <command_interface name="acceleration"/> -->
         <state_interface name="velocity" />
-        <state_interface name="effort" />
+        <!-- <state_interface name="acceleration" /> -->
       </joint>
       <joint name="${tf_prefix}${gripper_name}_l_finger_joint">
@@ -59,11 +60,12 @@
           <command_interface name="position" />
           <command_interface name="velocity"/>
-          <command_interface name="effort"/>
+          <!-- <command_interface name="acceleration"/> -->
           <state_interface name="position" />
           <state_interface name="velocity" />
-          <state_interface name="effort" />
+          <!-- <state_interface name="acceleration" /> -->
         </xacro:unless>
       </joint>
     </ros2_control>
+    <xacro:rbs_gripper_transmission joint_name="${tf_prefix}${gripper_name}_rot_base_joint" />
   </xacro:macro>
 </robot>
